Commit message: Updated project files

File: src/robot_description/urdf/web_robot.urdf.xacro (robot description, xacro)
@@ -3,13 +3,17 @@
   <xacro:arg name="mesh_package" default="robot_description"/>
   <xacro:arg name="mesh_scale" default="0.1 0.1 0.1"/>
-  <xacro:arg name="wheel_mass" default="0.5"/>
+  <xacro:arg name="wheel_mass" default="0.25"/>
   <xacro:arg name="base_mass" default="2.0"/>
+  <xacro:arg name="pi" default="3.141592653589793"/>
   <material name="blue"><color rgba="0 0 0.8 1"/></material>
   <material name="black"><color rgba="0 0 0 1"/></material>
   <material name="white"><color rgba="1 1 1 1"/></material>
+  <physics type="ode">
+    <real_time_update_rate>100</real_time_update_rate>
+  </physics>
     <!-- Define inertial property macros  -->
   <xacro:macro name="box_inertia" params="m w h d">
     <inertial>
-      <origin xyz="0 0 0" rpy="${pi/2} 0 ${pi/2}"/>
+      <origin xyz="0 0 -0.05" rpy="0 0 0"/>
       <mass value="${m}"/>
       <inertia ixx="${(m/12) * (h*h + d*d)}" ixy="0.0" ixz="0.0" iyy="${(m/12) * (w*w + d*d)}" iyz="0.0" izz="${(m/12) * (w*w + h*h)}"/>
@@ -44,11 +48,117 @@
         </geometry>
       </collision>
-      <inertial>
+      <xacro:box_inertia m="$(arg base_mass)" w="0.16" h="0.2" d="0.03"/>
+      <!-- <inertial>
         <mass value="$(arg base_mass)"/>
         <inertia ixx="0.0093" ixy="0.0" ixz="0.0"
                  iyy="0.0270" iyz="0.0" izz="0.0337"/>
-      </inertial>
+      </inertial> -->
     </link>
   </xacro:macro>
+  <!-- DRIVEN wheel macro (front wheels - high longitudinal grip) -->
+<xacro:macro name="driven_wheel_macro" params="name rpy xyz">
+  <link name="${name}">
+    <visual>
+      <origin rpy="${rpy}" xyz="0 0 0"/>
+      <geometry>
+        <mesh filename="package://$(arg mesh_package)/meshes/wheel.dae" scale="$(arg mesh_scale)"/>
+      </geometry>
+      <material name="black"/>
+    </visual>
+    <collision>
+      <origin rpy="${rpy}" xyz="0 0 0"/>
+      <geometry>
+        <mesh filename="package://$(arg mesh_package)/meshes/wheel.dae" scale="$(arg mesh_scale)"/>
+      </geometry>
+      <surface>
+        <friction>
+          <ode>
+            <mu>1.0</mu>       <!-- good forward grip -->
+            <mu2>0.003</mu2>     <!-- some lateral resistance is OK for driven wheels -->
+            <slip1>0.02</slip1>
+            <slip2>1.0</slip2>
+          </ode>
+        </friction>
+        <contact>
+          <ode>
+            <kp>100000.0</kp>
+            <kd>10.0</kd>
+            <min_depth>0.001</min_depth>
+          </ode>
+        </contact>
+      </surface>
+    </collision>
+    <xacro:cylinder_inertia m="$(arg wheel_mass)" r="0.054" h="0.02"/>
+  </link>
+  <joint name="${name}_joint" type="continuous">
+    <axis xyz="0 1 0"/>
+    <parent link="base_link"/>
+    <child link="${name}"/>
+    <origin rpy="0 0 0" xyz="${xyz}"/>
+  </joint>
+  <transmission name="${name}_trans">
+    <type>transmission_interface/SimpleTransmission</type>
+    <joint name="${name}_joint">
+      <hardware_interface>hardware_interface/VelocityJointInterface</hardware_interface>
+    </joint>
+    <actuator name="${name}_motor">
+      <hardware_interface>hardware_interface/VelocityJointInterface</hardware_interface>
+      <mechanicalReduction>1</mechanicalReduction>
+    </actuator>
+  </transmission>
+</xacro:macro>
+<!-- PASSIVE wheel macro (rear wheels - must slip laterally during rotation) -->
+<xacro:macro name="passive_wheel_macro" params="name rpy xyz ">
+  <link name="${name}">
+    <visual>
+      <origin rpy="${rpy}" xyz="0 0 0"/>
+      <geometry>
+        <mesh filename="package://$(arg mesh_package)/meshes/wheel.dae" scale="$(arg mesh_scale)"/>
+      </geometry>
+      <material name="black"/>
+    </visual>
+    <collision>
+      <origin rpy="${rpy}" xyz="0 0 0"/>
+      <geometry>
+        <mesh filename="package://$(arg mesh_package)/meshes/wheel.dae" scale="$(arg mesh_scale)"/>
+      </geometry>
+      <surface>
+        <friction>
+          <ode>
+            <mu>1.5</mu>       <!-- some forward grip to follow the robot -->
+            <mu2>0.01</mu2>    <!-- near-zero lateral friction = free sideways slip -->
+            <slip1>0.002</slip1>
+            <slip2>1.01</slip2> <!-- max lateral slip allowed -->
+          </ode>
+        </friction>
+        <contact>
+          <ode>
+            <kp>100000.0</kp>
+            <kd>10.0</kd>
+            <min_depth>0.001</min_depth>
+          </ode>
+        </contact>
+      </surface>
+    </collision>
+    <xacro:cylinder_inertia m="$(arg wheel_mass)" r="0.054" h="0.02"/>
+  </link>
+  <joint name="${name}_joint" type="continuous">
+    <axis xyz="0 1 0"/>
+    <parent link="base_link"/>
+    <child link="${name}"/>
+    <origin rpy="0 0 0" xyz="${xyz}"/>
+  </joint>
+  <transmission name="${name}_trans">
+    <type>transmission_interface/SimpleTransmission</type>
+    <joint name="${name}_joint">
+      <hardware_interface>hardware_interface/VelocityJointInterface</hardware_interface>
+    </joint>
+    <actuator name="${name}_motor">
+      <hardware_interface>hardware_interface/VelocityJointInterface</hardware_interface>
+      <mechanicalReduction>1</mechanicalReduction>
+    </actuator>
+  </transmission>
+</xacro:macro>
+<!--
   <xacro:macro name="wheel_macro" params="name rpy xyz">
     <link name="${name}">
@@ -60,23 +170,25 @@
         <material name="black"/>
       </visual>
-      <collision>
-        <origin rpy="${rpy}" xyz="0 0 0"/>
-        <geometry>
-          <mesh filename="package://$(arg mesh_package)/meshes/wheel.dae" scale="$(arg mesh_scale)" />
-        </geometry>
-         <surface>
-          <friction>
-            <ode>
-              <mu>0.8</mu>
-              <mu2>0.8</mu2>
-            </ode>
-          </friction>
-        </surface>
-      </collision>
-      <inertial>
-        <mass value="$(arg wheel_mass)"/>
-        <inertia ixx="0.000125" ixy="0.0" ixz="0.0"
-                 iyy="0.000245" iyz="0.0" izz="0.000125"/>
-      </inertial>
+     <collision>
+      <origin rpy="${rpy}" xyz="0 0 0"/>
+      <geometry>
+        <cylinder radius="0.054" length="0.02"/>
+      </geometry>
+      <surface>
+        <friction>
+          <ode>
+            <mu>0.5</mu>   <mu2>0.01</mu2>
+            <slip1>0.01</slip1>
+            <slip2>1.0</slip2>  </ode>
+        </friction>
+        <contact>
+          <ode>
+            <kp>1000000.0</kp>
+            <kd>10.0</kd>     <min_depth>0.001</min_depth>
+          </ode>
+        </contact>
+      </surface>
+    </collision>
+      <xacro:cylinder_inertia m="$(arg wheel_mass)" r="0.054" h="0.02"/>
     </link>
     <joint name="${name}_joint" type="continuous">
@@ -100,13 +212,13 @@
       </actuator>
     </transmission>
-  </xacro:macro>
+  </xacro:macro> -->
   <xacro:base_link_macro name="base_link"/>
-  <!-- Dummy footprint
+  <!-- Dummy footprint -->
   <link name="base_footprint"/>
   <joint name="base_link_joint" type="fixed">
     <parent link="base_footprint"/>
     <child link="base_link"/>
-    <origin xyz="0 0 0" rpy="0 0 0"/>
-  </joint> -->
+    <origin xyz="0 0 0.1" rpy="0 0 0"/>
+  </joint>
   <link name="camera_cad">
     <visual>
@@ -145,13 +257,21 @@
     <origin xyz="0.0 -0.05 0.095" rpy="0 0 1.57075"/>
   </joint>
+<!-- Front wheels: DRIVEN (controlled by diff_drive_controller) -->
+<xacro:driven_wheel_macro  name="front_right_wheel" rpy="-1.57075 0 0" xyz="-0.069 -0.102 0.054"/>
+<xacro:driven_wheel_macro  name="front_left_wheel"  rpy="1.57075 0 0"  xyz="-0.069 0.1 0.054"/>
+<!-- Rear wheels: PASSIVE (free to slip sideways during turns) -->
+<xacro:passive_wheel_macro name="back_right_wheel"  rpy="-1.57075 0 0" xyz="0.069 -0.102 0.054"/>
+<xacro:passive_wheel_macro name="back_left_wheel"   rpy="1.57075 0 0"  xyz="0.069 0.1 0.054"/>
+<!--
   <xacro:wheel_macro name="front_right_wheel" rpy="-1.57075 0 0" xyz="-0.069 -0.102 0.054"/>
   <xacro:wheel_macro name="front_left_wheel"  rpy="1.57075 0 0"  xyz="-0.069 0.1 0.054"/>
   <xacro:wheel_macro name="back_right_wheel"  rpy="-1.57075 0 0" xyz="0.069 -0.102 0.054"/>
-  <xacro:wheel_macro name="back_left_wheel"   rpy="1.57075 0 0"  xyz="0.069 0.1 0.054"/>
+  <xacro:wheel_macro name="back_left_wheel"   rpy="1.57075 0 0"  xyz="0.069 0.1 0.054"/> -->
+  <!-- Right side wheels (rpy has -1.57) -->
   <gazebo>
     <plugin name="gazebo_ros2_control" filename="libgazebo_ros2_control.so" >
-      <robot_param>robot_description</robot_param>
+      <!-- <robot_param>robot_description</robot_param>
       <robotNamespace>web_robot</robotNamespace>
-      <robotSimType>gazebo_ros2_control/GazeboSystem</robotSimType>
+      <robotSimType>gazebo_ros2_control/GazeboSystem</robotSimType> -->
       <parameters>$(find robot_description)/config/diff_drive_controllers.yaml</parameters>
     </plugin>
@@ -234,5 +354,6 @@
     <pose>0 0 0 0 0 0</pose>
     <visualize>true</visualize>
-    <update_rate>10.0</update_rate>
+    <update_rate>60.0</update_rate>
+    <output_type>sensor_msgs/LaserScan</output_type>
     <ray>
       <scan>
@@ -253,10 +374,10 @@
       <ros>
         <namespace>/</namespace>
-        <remapping>~/out:=scan</remapping>
+        <remapping>~/out:=scan_laser</remapping>
       </ros>
       <!-- <output_type>sensor_msgs/msg/LaserScan</output_type>
       <radiation_type>laser</radiation_type> -->
       <frame_name>laser_link</frame_name>
-      <topic_name>scan</topic_name>
+      <topic_name>scan_laser</topic_name>
     </plugin>
   </sensor>
@@ -284,5 +405,5 @@
    <plugin filename="libgazebo_ros_imu_sensor.so" name="imu_plugin">
       <ros>
-        <!-- <namespace>/demo</namespace> -->
+        <namespace>/</namespace>
         <remapping>~/out:=imu</remapping>
       </ros>
@@ -290,5 +411,5 @@
     </plugin>
     <always_on>true</always_on>
-    <update_rate>100</update_rate>
+    <update_rate>100.0</update_rate>
     <visualize>true</visualize>
     <imu>
